File: pcb/PDU_Meanwell_LRS.brd (EAGLE design)
At the start: 41.5 x 80 mm, 13 parts, among them J1 TERMINAL-1X02-5.08, X1 XT60-PW-F, X2 XT60-PW-F, X3 XT60-PW-F

Commit message: Initial commit
Parts:
- added U$1: (no value), M2M-Frames:BERGDAHL-20MM-TPLACE
- added U$2: (no value), M2M-Frames:OSHW-5MM-TPLACE
- added U$3: (no value), M2M-Frames:BERGDAHL-20MM-BPLACE
- added U$4: (no value), M2M-Frames:OSHW-8MM-BPLACE
- moved R1 4.30 mm to (14.0, 71.5), turned to 180 degrees
- moved J1 0.78 mm to (35.3, 39.9), turned to 0 degrees
- moved F1 0.50 mm to (24.5, 40.0)
- moved F2 0.50 mm to (24.4, 16.5)
- moved F3 0.50 mm to (24.5, 64.0)
- moved H1 0.50 mm to (35.0, 6.00)
- moved H2 0.50 mm to (35.0, 74.0)
- turned D1 to 180 degrees
Routing:
- net VCC: track 0.00 -> 10.2 mm
- net GND: track 6.38 -> 0.00 mm, vias 0 -> 19
- net N$3: track 6.87 -> 2.67 mm
- added copper zone on layer 1, net GND
Other:
- board size 41.5 x 80 mm -> 41 x 80 mm
- board text added: "2023-05-27"
- board text added: "GND"
- board text added: "LRS PDU"
- board text added: "VCC"
